File: Electronics/Final version/WiFi Module/WiFi_Module.brd (EAGLE design)
At the start: 35 x 32 mm, 10 parts

Commit message: ASD
Connections:
- removed net ARDUINO5V: INPUT-3V3.3
- new net VIN: INPUT-3V3.2
- net GND: now also INPUT-3V3.3; no longer INPUT-3V3.2
Routing:
- net GND: track 55.7 -> 55.0 mm
Changed lines of the file:
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@@
 <autorouter>
 <pass name="Default">
-<param name="RoutingGrid" value="50mil"/>
+<param name="RoutingGrid" value="6.25mil"/>
 <param name="AutoGrid" value="1"/>
 <param name="Efforts" value="2"/>
 <param name="TopRouterVariant" value="1"/>
 <param name="tpViaShape" value="round"/>
-<param name="PrefDir.1" value="a"/>
+<param name="PrefDir.1" value="*"/>
 <param name="PrefDir.2" value="0"/>
 <param name="PrefDir.3" value="0"/>
@@
 <param name="PrefDir.14" value="0"/>
 <param name="PrefDir.15" value="0"/>
-<param name="PrefDir.16" value="a"/>
+<param name="PrefDir.16" value="-"/>
 <param name="cfVia" value="8"/>
 <param name="cfNonPref" value="5"/>
@@
 <wire x1="23.4696" y1="30.1752" x2="21.0312" y2="30.1752" width="0.1524" layer="1"/>
 <wire x1="21.0312" y1="30.1752" x2="21.014" y2="30.054" width="0.1524" layer="1"/>
-<wire x1="23.4696" y1="30.1752" x2="23.561" y2="30.181" width="0.1524" layer="1"/>
 <wire x1="23.4696" y1="30.1752" x2="23.4696" y2="26.8224" width="0.1524" layer="1"/>
 <wire x1="23.4696" y1="26.8224" x2="23.516" y2="26.715" width="0.1524" layer="1"/>
@@
 <contactref element="U1" pad="GND"/>
 <contactref element="FLASH" pad="P$2"/>
-<contactref element="INPUT-3V3" pad="2"/>
 <contactref element="RESET" pad="P$2"/>
 <contactref element="R4" pad="1"/>
+<contactref element="INPUT-3V3" pad="3"/>
 <wire x1="15.8496" y1="17.9832" x2="15.8496" y2="26.5176" width="0.1524" layer="16"/>
 <wire x1="10.2108" y1="12.3444" x2="15.8496" y2="17.9832" width="0.1524" layer="16"/>
@@
 <wire x1="15.8496" y1="26.5176" x2="15.917" y2="26.588" width="0.1524" layer="16"/>
 <wire x1="11.2776" y1="9.6012" x2="11.376" y2="9.483" width="0.1524" layer="16"/>
-<wire x1="16.764" y1="2.8956" x2="21.336" y2="2.8956" width="0.1524" layer="1"/>
+<wire x1="19.3548" y1="2.8956" x2="21.336" y2="2.8956" width="0.1524" layer="1"/>
 <wire x1="21.336" y1="2.8956" x2="23.0124" y2="2.8956" width="0.1524" layer="1"/>
-<wire x1="14.0208" y1="5.6388" x2="16.764" y2="2.8956" width="0.1524" layer="1"/>
+<wire x1="16.6116" y1="5.6388" x2="19.3548" y2="2.8956" width="0.1524" layer="1"/>
 <wire x1="23.0124" y1="2.8956" x2="23.079" y2="2.774" width="0.1524" layer="1"/>
-<wire x1="14.0208" y1="5.6388" x2="13.984" y2="5.736" width="0.1524" layer="1"/>
+<wire x1="16.6116" y1="5.6388" x2="16.524" y2="5.736" width="0.1524" layer="1"/>
 <wire x1="24.8412" y1="6.096" x2="28.3464" y2="6.096" width="0.1524" layer="1"/>
 <wire x1="24.384" y1="5.6388" x2="24.8412" y2="6.096" width="0.1524" layer="1"/>
@@
 <wire x1="28.4988" y1="15.5448" x2="28.4226" y2="15.6924" width="0.1524" layer="1"/>
 <wire x1="28.4988" y1="6.2484" x2="28.46" y2="6.2214" width="0.1524" layer="1"/>
-<wire x1="11.43" y1="8.2296" x2="11.43" y2="9.4488" width="0.1524" layer="1"/>
-<wire x1="13.8684" y1="5.7912" x2="11.43" y2="8.2296" width="0.1524" layer="1"/>
+<wire x1="12.8016" y1="9.4488" x2="11.43" y2="9.4488" width="0.1524" layer="1"/>
+<wire x1="16.4592" y1="5.7912" x2="12.8016" y2="9.4488" width="0.1524" layer="1"/>
 <wire x1="11.43" y1="9.4488" x2="11.376" y2="9.483" width="0.1524" layer="1"/>
-<wire x1="13.8684" y1="5.7912" x2="13.984" y2="5.736" width="0.1524" layer="1"/>
+<wire x1="16.4592" y1="5.7912" x2="16.524" y2="5.736" width="0.1524" layer="1"/>
 </signal>
 <signal name="N$3">
@@
 <wire x1="28.6512" y1="26.67" x2="28.596" y2="26.715" width="0.1524" layer="1"/>
 <wire x1="33.0708" y1="22.2504" x2="32.9226" y2="22.1924" width="0.1524" layer="1"/>
-</signal>
-<signal name="ARDUINO5V">
-<contactref element="INPUT-3V3" pad="3"/>
 </signal>
 <signal name="EN">
@@
 <wire x1="8.6868" y1="29.2608" x2="8.549" y2="29.349" width="0.1524" layer="1"/>
 </signal>
+<signal name="VIN">
+<contactref element="INPUT-3V3" pad="2"/>
+</signal>
 </signals>
